Commit message: added test model and config to rl inference

File: kangaroo_mujoco/models/mjcf_data_4dof_fake-forearm/robot_description_formatted.urdf (robot description, URDF)
Before this commit: robot kangaroo, 50 links, 49 joints
Links:
- added link imu_link; visual box size=0.01 0.01 0.01
- link leg_left_knee_link: geometry 
- link leg_right_knee_link: geometry 
Joints:
- added joint imu_joint: type fixed, parent torso_link, child imu_link, origin xyz=0.071 -0.0014 0.02 rpy=3.141592653589793 0.0 -1.5707963267948966

Commit message: updated model

File: kangaroo_mujoco/models/mjcf_data_4dof_fake-forearm/robot_description_formatted.urdf (robot description, URDF)
Before this commit: robot kangaroo, 51 links, 50 joints
Links:
- link leg_left_femur_link: geometry visual mesh filename=full/leg_4_collision_link.obj
- link leg_left_knee_link: geometry visual mesh filename=full/leg_tibia_link.obj
- link leg_right_femur_link: geometry visual mesh filename=full/leg_4_collision_link.obj
- link leg_right_knee_link: geometry visual mesh filename=full/leg_tibia_link.obj
