Commit message: Update to new ankle configuration data

File: kangaroo_mujoco/models/mjcf_data_floating_no-arm_no-end-effector_no-end-effector_detachable_empty/robot_description_formatted.urdf (robot description, URDF)
Before this commit: robot kangaroo, 94 links, 93 joints
Links:
- removed link left_foot_ft
- removed link right_foot_ft
- added link ankle_left_ft_sensor_link, mass 0.345; visual mesh filename=full/foot-ft.obj
- added link ankle_right_ft_sensor_link, mass 0.345; visual mesh filename=full/foot-ft.obj
- link arm_cover_left_cover_link: geometry visual mesh filename=full/arm_cover_link.obj
- link arm_cover_right_cover_link: geometry visual mesh filename=full/arm_cover_link.obj
- link back_handle: geometry visual mesh filename=full/handle.obj
- link base_link: geometry visual mesh filename=full/base_link_with_pelvis.obj
- link left_foot: mass 0.126216116323818 -> 0.170698
- link left_foot_sole: mass 0.34359589794105 -> 1.081199
- link leg_left_1_link: geometry visual mesh filename=full/leg_left_1_link.obj scale=1 1 1
- link leg_left_2_link: geometry visual mesh filename=full/leg_left_2_link.obj scale=1 1 1
- link leg_left_3_link: geometry visual mesh filename=full/leg_left_3_link.obj scale=1 1 1
- link leg_left_4_link: mass 0.094024 -> 0.132674
- link leg_left_femur_link: geometry visual mesh filename=full/leg_4_collision_link.obj
- link leg_left_knee_link: geometry visual mesh filename=full/leg_tibia_link.obj
- link leg_right_1_link: geometry visual mesh filename=full/leg_right_1_link.obj scale=1 1 1
- link leg_right_2_link: geometry visual mesh filename=full/leg_right_2_link.obj scale=1 1 1
- link leg_right_3_link: geometry visual mesh filename=full/leg_right_3_link.obj scale=1 1 1
- link leg_right_4_link: mass 0.094024 -> 0.132674
- link leg_right_femur_link: geometry visual mesh filename=full/leg_4_collision_link.obj
- link leg_right_knee_link: geometry visual mesh filename=full/leg_tibia_link.obj
- link pelvis_1_link: geometry visual mesh filename=full/pelvis_1_link.obj
- link pelvis_2_link: geometry visual mesh filename=full/pelvis_2_link.obj
- link pelvis_base_link: geometry visual mesh filename=full/pelvis_base_link.obj
- link right_foot: mass 0.126216116323818 -> 0.170698
- link right_foot_sole: mass 0.34359589794105 -> 1.081199
- link torso_front_down_rgbd_camera_link: geometry visual mesh filename=full/d435.obj
- link torso_front_up_rgbd_camera_link: geometry visual mesh filename=full/d435.obj
- link torso_link: geometry visual mesh filename=full/torso_link.obj
- link torso_rear_down_rgbd_camera_link: geometry visual mesh filename=full/d435.obj
- link torso_rear_up_rgbd_camera_link: geometry visual mesh filename=full/d435.obj
Joints:
- joint left_foot_ft: child left_foot_ft -> ankle_left_ft_sensor_link; origin xyz=0 0 0.014 rpy=0 3.1416 0 -> xyz=0 0 -0.014 rpy=0 0 3.141592653589793
- joint left_foot_joint: origin xyz=0.0 0.0 0 rpy=0 0 0 -> xyz=0 0 0 rpy=0 0 0
- joint left_foot_sole: origin xyz=0 0 -0.038472 rpy=0 3.1416 0 -> xyz=0 0 -0.053972 rpy=0 0 -3.141592653589793; parent left_foot_ft -> ankle_left_ft_sensor_link
- joint leg_left_4_joint: axis 0 -1 0 -> 0 1 0; origin xyz=0 0 0 rpy=0 -0.3490658503988659 3.1416 -> xyz=0.0 0 0.0 rpy=0 3.141592653589793 0
- joint leg_left_5_joint: origin xyz=0 0 0 rpy=0 0 0 -> xyz=0 0 0 rpy=0 0.3490658503988659 0
- joint leg_left_ankle_attach_joint: origin xyz=0.013168 0 0.036178 rpy=0 0.34907 0 -> xyz=0.013168 0 -0.036178 rpy=0 -0.3490658503988659 0
- joint leg_right_4_joint: axis 0 -1 0 -> 0 1 0; origin xyz=0 0 0 rpy=0 -0.3490658503988659 3.1416 -> xyz=0.0 0 0.0 rpy=0 3.141592653589793 0
- joint leg_right_5_joint: origin xyz=0 0 0 rpy=0 0 0 -> xyz=0 0 0 rpy=0 0.3490658503988659 0
- joint leg_right_ankle_attach_joint: origin xyz=0.013168 0 0.036178 rpy=0 0.34907 0 -> xyz=0.013168 0 -0.036178 rpy=0 -0.3490658503988659 0
- joint right_foot_ft: child right_foot_ft -> ankle_right_ft_sensor_link; origin xyz=0 0 0.014 rpy=0 3.1416 0 -> xyz=0 0 -0.014 rpy=0 0 3.141592653589793
- joint right_foot_joint: origin xyz=0.0 0.0 0 rpy=0 0 0 -> xyz=0 0 0 rpy=0 0 0
- joint right_foot_sole: origin xyz=0 0 -0.038472 rpy=0 3.1416 0 -> xyz=0 0 -0.053972 rpy=0 0 -3.141592653589793; parent right_foot_ft -> ankle_right_ft_sensor_link
