Commit message: Fix renamed links from *_foot_sole to *_sole_link

File: kangaroo_mujoco/models/mjcf_data_fixed_no-arm_no-end-effector_no-end-effector_detachable_empty/robot_description_formatted.urdf (robot description, URDF)
Before this commit: robot kangaroo, 93 links, 92 joints
Links:
- removed link left_foot_sole
- removed link right_foot_sole
- added link left_sole_link, mass 1.081199; visual mesh filename=full/foot-sole.obj
- added link right_sole_link, mass 1.081199; visual mesh filename=full/foot-sole.obj
Joints:
- removed joint left_foot_sole
- removed joint right_foot_sole
- added joint left_sole_link: type fixed, parent ankle_left_ft_sensor_link, child left_sole_link, origin xyz=0 0 -0.053972 rpy=0 0 -3.141592653589793, axis 0 0 0
- added joint right_sole_link: type fixed, parent ankle_right_ft_sensor_link, child right_sole_link, origin xyz=0 0 -0.053972 rpy=0 0 -3.141592653589793, axis 0 0 0

File: kangaroo_mujoco/models/mjcf_data_floating_no-arm_no-end-effector_no-end-effector_detachable_empty/robot_description_formatted.urdf (robot description, URDF)
Before this commit: robot kangaroo, 94 links, 93 joints
Links:
- removed link left_foot_sole
- removed link right_foot_sole
- added link left_sole_link, mass 1.081199; visual mesh filename=full/foot-sole.obj
- added link right_sole_link, mass 1.081199; visual mesh filename=full/foot-sole.obj
Joints:
- removed joint left_foot_sole
- removed joint right_foot_sole
- added joint left_sole_link: type fixed, parent ankle_left_ft_sensor_link, child left_sole_link, origin xyz=0 0 -0.053972 rpy=0 0 -3.141592653589793, axis 0 0 0
- added joint right_sole_link: type fixed, parent ankle_right_ft_sensor_link, child right_sole_link, origin xyz=0 0 -0.053972 rpy=0 0 -3.141592653589793, axis 0 0 0

File: kangaroo_mujoco/models/mjcf_data_floating_no-arm_no-end-effector_no-end-effector_detachable_stairs/robot_description_formatted.urdf (robot description, URDF)
Before this commit: robot kangaroo, 94 links, 93 joints
Links:
- removed link left_foot_sole
- removed link right_foot_sole
- added link left_sole_link, mass 0.34359589794105; visual mesh filename=full/foot-sole.obj
- added link right_sole_link, mass 0.34359589794105; visual mesh filename=full/foot-sole.obj
Joints:
- removed joint left_foot_sole
- removed joint right_foot_sole
- added joint left_sole_link: type fixed, parent left_foot_ft, child left_sole_link, origin xyz=0 0 -0.038472 rpy=0 3.1416 0, axis 0 0 0
- added joint right_sole_link: type fixed, parent right_foot_ft, child right_sole_link, origin xyz=0 0 -0.038472 rpy=0 3.1416 0, axis 0 0 0
